Commit message: Update Classic and Si tool URDF

File: urdf/include/classic/tool.macro.xacro (robot description, xacro)
@@ -4,19 +4,46 @@
     <!-- Macro for the 8mm Small Clip Applier (sca) tool -->
     <xacro:macro name="tool_sca_8mm" params="prefix parent_link xyz:='0 0 0' rpy:='0 0 0'">
-        <xacro:tool_shaft prefix="${prefix}" diameter="8mm" parent_link="${parent_link}" xyz="${xyz}" rpy="${rpy}"/>
-        <xacro:tool_wrist_8mm prefix="${prefix}" parent_link="${prefix}tool_wrist_mount_link"/>
-        <xacro:tool_gripper_sca_8mm prefix="${prefix}" parent_link="${prefix}tool_gripper_mount_link"/>
+        <xacro:tool_shaft
+            prefix="${prefix}"
+            diameter="8mm"
+            parent_link="${parent_link}"
+            xyz="${xyz}"
+            rpy="${rpy}"/>
+        <xacro:tool_wrist_8mm
+            prefix="${prefix}"
+            parent_link="${prefix}tool_wrist_mount_link"/>
+        <xacro:tool_gripper_sca_8mm
+            prefix="${prefix}"
+            parent_link="${prefix}tool_gripper_mount_link"/>
     </xacro:macro>
     <!-- Macro for the 8mm Cadiere Forceps (cadiere) tool -->
     <xacro:macro name="tool_cadiere_8mm" params="prefix parent_link xyz:='0 0 0' rpy:='0 0 0'">
-        <xacro:tool_shaft prefix="${prefix}" diameter="8mm" parent_link="${parent_link}" xyz="${xyz}" rpy="${rpy}"/>
-        <xacro:tool_wrist_8mm prefix="${prefix}" parent_link="${prefix}tool_wrist_mount_link"/>
-        <xacro:tool_gripper_cadiere_8mm prefix="${prefix}" parent_link="${prefix}tool_gripper_mount_link"/>
+        <xacro:tool_shaft
+            prefix="${prefix}"
+            diameter="8mm"
+            parent_link="${parent_link}"
+            xyz="${xyz}"
+            rpy="${rpy}"/>
+        <xacro:tool_wrist_8mm
+            prefix="${prefix}"
+            parent_link="${prefix}tool_wrist_mount_link"/>
+        <xacro:tool_gripper_cadiere_8mm
+            prefix="${prefix}"
+            parent_link="${prefix}tool_gripper_mount_link"/>
     </xacro:macro>
     <!-- Macro for the 5mm Round Tip Scissors (rts) tool -->
     <xacro:macro name="tool_rts_5mm" params="prefix parent_link xyz:='0 0 0' rpy:='0 0 0'">
-        <xacro:tool_shaft prefix="${prefix}" diameter="5mm" parent_link="${parent_link}" xyz="${xyz}" rpy="${rpy}"/>
-        <xacro:tool_wrist_5mm prefix="${prefix}" parent_link="${prefix}tool_wrist_mount_link"/>
-        <xacro:tool_gripper_rts_5mm prefix="${prefix}" parent_link="${prefix}tool_gripper_mount_link"/>
+        <xacro:tool_shaft
+            prefix="${prefix}"
+            diameter="5mm"
+            parent_link="${parent_link}"
+            xyz="${xyz}"
+            rpy="${rpy}"/>
+        <xacro:tool_wrist_5mm
+            prefix="${prefix}"
+            parent_link="${prefix}tool_wrist_mount_link"/>
+        <xacro:tool_gripper_rts_5mm
+            prefix="${prefix}"
+            parent_link="${prefix}tool_gripper_mount_link"/>
     </xacro:macro>
     <!-- Macro for tool shaft (8mm and 5mm)  -->

File: urdf/include/si/tool.macro.xacro (robot description, xacro)
@@ -2,36 +2,4 @@
 <robot xmlns:xacro="http://www.ros.org/wiki/xacro">
     <xacro:include filename="$(find dvrk_description)/urdf/include/colors.xacro"/>
-    <!-- Macro for a tool -->
-    <xacro:macro name="tool" params="prefix tool parent_link xyz:='0 0 0' rpy:='0 0 0'">
-        <!-- camera -->
-        <xacro:if value="${tool == 'camera'}">
-        </xacro:if>
-        <!-- large needle driver -->
-        <xacro:if value="${tool == 'lnd_8mm'}">
-        </xacro:if>
-    </xacro:macro>
-    <!-- Macro for camera -->
-    <xacro:macro name="tool_camera" params="prefix parent_link xyz:='0 0 0' rpy:='0 0 0'">
-        <link name="${prefix}tool_base_link"/>
-        <link name="${prefix}tool_camera_link">
-            <visual>
-                <origin xyz="0 0 0" rpy="0 0 ${pi}"/>
-                <geometry>
-                    <mesh filename="package://dvrk_description/meshes/si/tool/camera.stl"/>
-                </geometry>
-                <material name="DaVinciDarkGray"/>
-            </visual>
-        </link>
-        <joint name="${prefix}tool_base_joint" type="fixed">
-            <parent link="${parent_link}"/>
-            <child link="${prefix}tool_base_link"/>
-            <origin xyz="${xyz}" rpy="${rpy}"/>
-        </joint>
-        <joint name="${prefix}tool_camera_joint" type="fixed">
-            <parent link="${prefix}tool_base_link"/>
-            <child link="${prefix}tool_camera_link"/>
-            <origin xyz="0 ${-0.05591+0.0267} 0" rpy="0 0 0"/>
-        </joint>
-    </xacro:macro>
     <!-- Macro for 8mm large needle driver -->
     <xacro:macro name="tool_lnd_8mm" params="prefix parent_link xyz:='0 0 0' rpy:='0 0 0'">
@@ -97,4 +65,10 @@
                 <material name="DaVinciMetallic"/>
             </visual>
+            <collision>
+                <origin xyz="0 0 0" rpy="0 0 ${-pi/2}"/>
+                <geometry>
+                    <mesh filename="package://dvrk_description/meshes/si/tool/wrist_8mm/roll.stl"/>
+                </geometry>
+            </collision>
         </link>
         <link name="${prefix}tool_wrist_pitch_shaft_link">
@@ -106,4 +80,10 @@
                 <material name="DaVinciMetallic"/>
             </visual>
+            <collision></collision>
+                <origin xyz="0 0 0" rpy="0 0 ${-pi/2}"/>
+                <geometry>
+                    <mesh filename="package://dvrk_description/meshes/si/tool/wrist_8mm/pitch_shaft.stl"/>
+                </geometry>
+            </collision>
         </link>
         <link name="${prefix}tool_wrist_pitch_link">
@@ -115,4 +95,10 @@
                 <material name="DaVinciMetallic"/>
             </visual>
+            <collision></collision>
+                <origin xyz="0 0 0" rpy="${-pi/2} 0 ${-pi/2}"/>
+                <geometry>
+                    <mesh filename="package://dvrk_description/meshes/si/tool/wrist_8mm/pitch.stl"/>
+                </geometry>
+            </collision>
         </link>
         <link name="${prefix}tool_wrist_yaw_link">
@@ -124,4 +110,10 @@
                 <material name="DaVinciMetallic"/>
             </visual>
+            <collision>
+                <origin xyz="0 0 0" rpy="0 ${pi/2} 0"/>
+                <geometry>
+                    <mesh filename="package://dvrk_description/meshes/si/tool/wrist_8mm/yaw.stl"/>
+                </geometry>
+            </collision>
         </link>
         <!-- 8mm wrist joints -->
@@ -172,4 +164,10 @@
                 <material name="DaVinciMetallic"/>
             </visual>
+            <collision>
+                <origin xyz="0 0 0" rpy="${pi} ${-pi/2} 0"/>
+                <geometry>
+                    <mesh filename="package://dvrk_description/meshes/si/tool/gripper_lnd_8mm.stl"/>
+                </geometry>
+            </collision>
         </link>
         <link name="${prefix}tool_gripper2_link">
@@ -181,4 +179,10 @@
                 <material name="DaVinciMetallic"/>
             </visual>
+            <collision>
+                <origin xyz="0 0 0" rpy="${pi} ${-pi/2} 0"/>
+                <geometry>
+                    <mesh filename="package://dvrk_description/meshes/si/tool/gripper_lnd_8mm.stl"/>
+                </geometry>
+            </collision>
         </link>
         <joint name="${prefix}tool_gripper_root_joint" type="fixed">
@@ -187,5 +191,5 @@
             <origin xyz="${xyz}" rpy="${rpy}"/>
         </joint>
-        <joint name="${prefix}tool_gripper1_joint" type="revolute">
+        <joint name="${prefix}tool_jaw_joint" type="revolute">
             <parent link="${prefix}tool_gripper_root_link"/>
             <child link="${prefix}tool_gripper1_link"/>
@@ -194,10 +198,10 @@
             <limit lower="0" upper="1" effort="5" velocity="1"/>
         </joint>
-        <joint name="${prefix}tool_gripper2_mimic_joint" type="revolute">
+        <joint name="${prefix}tool_jaw_mimic_joint" type="revolute">
             <parent link="${parent_link}"/>
             <child link="${prefix}tool_gripper2_link"/>
             <origin xyz="${xyz}" rpy="${pi} 0 0"/>
             <axis xyz="0 0 1"/>
-            <mimic joint="${prefix}tool_gripper1_joint" multiplier="1"/>
+            <mimic joint="${prefix}tool_jaw_joint" multiplier="1"/>
             <limit lower="0" upper="1" effort="5" velocity="1"/>
         </joint>
