Commit message: Streamline PSM Classic URDF

File: urdf/include/classic/psm.macro.xacro (robot description, xacro)
@@ -2,22 +2,7 @@
 <robot xmlns:xacro="http://www.ros.org/wiki/xacro">
     <xacro:include filename="$(find dvrk_description)/urdf/include/colors.xacro"/>
-    <!-- Macro for tools can be mounted on the PSM -->
     <xacro:include filename="$(find dvrk_description)/urdf/include/classic/tool.macro.xacro"/>
-    <xacro:macro name="psm_tool" params="prefix tool parent_link">
-        <!-- 8mm Small Clip Applier -->
-        <xacro:if value="${tool == 'sca_8mm'}">
-            <xacro:tool_sca_8mm prefix="${prefix}" parent_link="${parent_link}"/>
-        </xacro:if>
-        <!-- 8mm Cadiere Forceps -->
-        <xacro:if value="${tool == 'cadiere_8mm'}">
-            <xacro:tool_cadiere_8mm prefix="${prefix}" parent_link="${parent_link}"/>
-        </xacro:if>
-        <!-- 5mm Round Tip Scissors -->
-        <xacro:if value="${tool == 'rts_5mm'}">
-            <xacro:tool_rts_5mm prefix="${prefix}" parent_link="${parent_link}"/>
-        </xacro:if>
-    </xacro:macro>
     <!-- Macro for a complete PSM with tool -->
-    <xacro:macro name="psm" params="prefix color:='DaVinciOrange' show_RCM:='false' tool parent_link xyz:='0 0 0' rpy:='0 0 0'">
+    <xacro:macro name="psm" params="prefix color:='DaVinciOrange' show_RCM:='false' tool:='sca_8mm' parent_link xyz:='0 0 0' rpy:='0 0 0'">
         <xacro:psm_arm
             prefix="${prefix}"
@@ -27,5 +12,22 @@
             xyz="${xyz}"
             rpy="${rpy}"/>
-        <xacro:psm_tool prefix="${prefix}" tool="${tool}" parent_link="${prefix}tool_mount_link"/>
+        <!-- 8mm Small Clip Applier -->
+        <xacro:if value="${tool == 'sca_8mm'}">
+            <xacro:tool_sca_8mm
+                prefix="${prefix}"
+                parent_link="${prefix}tool_mount_link"/>
+        </xacro:if>
+        <!-- 8mm Cadiere Forceps -->
+        <xacro:if value="${tool == 'cadiere_8mm'}">
+            <xacro:tool_cadiere_8mm
+                prefix="${prefix}"
+                parent_link="${prefix}tool_mount_link"/>
+        </xacro:if>
+        <!-- 5mm Round Tip Scissors -->
+        <xacro:if value="${tool == 'rts_5mm'}">
+            <xacro:tool_rts_5mm
+                prefix="${prefix}"
+                parent_link="${prefix}tool_mount_link"/>
+        </xacro:if>
     </xacro:macro>
     <!-- Macro for a PSM arm without tool -->

Commit message: Update PSM Classic meshes

File: urdf/include/classic/psm.macro.xacro (robot description, xacro)
@@ -178,5 +178,5 @@
                 <origin xyz="0 0 0" rpy="0 0 ${pi/2}" />
                 <geometry>
-                    <mesh filename="package://dvrk_description/meshes/classic/psm/insertion_tool_adaptor.stl" />
+                    <mesh filename="package://dvrk_description/meshes/classic/psm/insertion.stl" />
                 </geometry>
                 <material name="${color}"/>
@@ -185,5 +185,5 @@
                 <origin xyz="0 0 0" rpy="0 0 ${pi/2}" />
                 <geometry>
-                    <mesh filename="package://dvrk_description/meshes/classic/psm/insertion_tool_adaptor.stl" />
+                    <mesh filename="package://dvrk_description/meshes/classic/psm/insertion.stl" />
                 </geometry>
             </collision>
