Commit message: Fix RCM frame orientation

File: urdf/include/classic/ecm.macro.xacro (robot description, xacro)
@@ -264,5 +264,5 @@
         </link>
         <joint name="${prefix}RCM_joint" type="fixed">
-            <origin xyz="0.612599207482277 0 0.10159534323531" rpy="0 0 ${-pi/2}" />
+            <origin xyz="0.612599207482277 0 0.10159534323531" rpy="0 0 0" />
             <parent link="${prefix}base_link" />
             <child link="${prefix}RCM_link" />

Commit message: Add parameter to hide/show RCM for PSM and ECM (Classic)

File: urdf/include/classic/ecm.macro.xacro (robot description, xacro)
@@ -3,5 +3,5 @@
     <xacro:include filename="$(find dvrk_description)/urdf/include/colors.xacro"/>
     <!-- Macro for da Vinci Endoscope Camera Manipulator (ecm) -->
-    <xacro:macro name="ecm" params="prefix parent_link xyz:='0 0 0' rpy:='0 0 0'">
+    <xacro:macro name="ecm" params="prefix show_RCM:='false' parent_link xyz:='0 0 0' rpy:='0 0 0'">
         <!-- ECM links -->
         <link name="${prefix}base_link">
@@ -253,13 +253,15 @@
         <!-- virtual RCM frame -->
         <link name="${prefix}RCM_link">
-            <!-- <visual>
-                <origin xyz="0 0 0" rpy="0 0 0" />
-                <geometry>
-                    <sphere radius="0.01"/>
-                </geometry>
-                <material name="">
-                    <color rgba="1 0 0 1" />
-                </material>
-            </visual> -->
+            <xacro:if value="${show_RCM}">
+                <visual>
+                    <origin xyz="0 0 0" rpy="0 0 0" />
+                    <geometry>
+                        <sphere radius="0.01"/>
+                    </geometry>
+                    <material name="">
+                        <color rgba="1 0 0 1" />
+                    </material>
+                </visual>
+            </xacro:if>
         </link>
         <joint name="${prefix}RCM_joint" type="fixed">

File: urdf/include/classic/psm.macro.xacro (robot description, xacro)
@@ -19,10 +19,16 @@
     </xacro:macro>
     <!-- Macro for a complete PSM with tool -->
-    <xacro:macro name="psm" params="prefix color:='DaVinciOrange' tool parent_link xyz:='0 0 0' rpy:='0 0 0'">
-        <xacro:psm_arm prefix="${prefix}" color="${color}" parent_link="${parent_link}" xyz="${xyz}" rpy="${rpy}"/>
+    <xacro:macro name="psm" params="prefix color:='DaVinciOrange' show_RCM:='false' tool parent_link xyz:='0 0 0' rpy:='0 0 0'">
+        <xacro:psm_arm
+            prefix="${prefix}"
+            color="${color}"
+            show_RCM="${show_RCM}"
+            parent_link="${parent_link}"
+            xyz="${xyz}"
+            rpy="${rpy}"/>
         <xacro:psm_tool prefix="${prefix}" tool="${tool}" parent_link="${prefix}tool_mount_link"/>
     </xacro:macro>
     <!-- Macro for a PSM arm without tool -->
-    <xacro:macro name="psm_arm" params="prefix color:='DaVinciOrange' parent_link xyz:='0 0 0' rpy:='0 0 0'">
+    <xacro:macro name="psm_arm" params="prefix color:='DaVinciOrange' show_RCM:='false' parent_link xyz:='0 0 0' rpy:='0 0 0'">
         <!-- PSM arm links -->
         <link name="${prefix}base_link">
@@ -247,13 +253,15 @@
         <!-- virtual link indicating RCM pose -->
         <link name="${prefix}RCM_link">
-            <!-- <visual>
-                <origin xyz="0 0 0" rpy="0 0 0" />
-                <geometry>
-                    <sphere radius="0.01"/>
-                </geometry>
-                <material name="">
-                    <color rgba="1 0 0 1" />
-                </material>
-            </visual> -->
+            <xacro:if value="${show_RCM}">
+                <visual>
+                    <origin xyz="0 0 0" rpy="0 0 0" />
+                    <geometry>
+                        <sphere radius="0.01"/>
+                    </geometry>
+                    <material name="">
+                        <color rgba="1 0 0 1" />
+                    </material>
+                </visual>
+            </xacro:if>
         </link>
         <joint name="${prefix}RCM_joint" type="fixed">

Commit message: Update based on ECM Classic meshes changes

File: urdf/include/classic/ecm.macro.xacro (robot description, xacro)
@@ -165,9 +165,9 @@
             </inertial>
         </link>
-        <link name="${prefix}camera_link">
-            <visual>
-                <origin xyz="0 0 0" rpy="0 0 0" />
-                <geometry>
-                    <mesh filename="package://dvrk_description/meshes/classic/ecm/camera.stl" />
+        <link name="${prefix}endoscope_link">
+            <visual>
+                <origin xyz="0 0 0" rpy="0 0 0" />
+                <geometry>
+                    <mesh filename="package://dvrk_description/meshes/classic/ecm/endoscope.stl" />
                 </geometry>
                 <material name="DaVinciMedGray"/>
@@ -176,5 +176,5 @@
                 <origin xyz="0 0 0" rpy="0 0 0" />
                 <geometry>
-                    <mesh filename="package://dvrk_description/meshes/classic/ecm/camera.stl" />
+                    <mesh filename="package://dvrk_description/meshes/classic/ecm/endoscope.stl" />
                 </geometry>
             </collision>
@@ -271,9 +271,9 @@
             <axis xyz="0 0 0" />
         </joint>
-        <!-- tool tip frame -->
+        <!-- endoscope tip frame -->
         <link name="${prefix}tip_link"/>
         <joint name="${prefix}tip_joint" type="fixed">
             <origin xyz="0 0 0.37364" rpy="0 0 0" />
-            <parent link="${prefix}camera_link" />
+            <parent link="${prefix}endoscope_link" />
             <child link="${prefix}tip_link" />
             <axis xyz="0 0 0" />

Commit message: Update ECM Classic meshes

File: urdf/include/classic/ecm.macro.xacro (robot description, xacro)
@@ -145,16 +145,16 @@
             </inertial>
         </link>
-        <link name="${prefix}camera_mount_link">
-            <visual>
-                <origin xyz="0 0 0" rpy="0 0 0" />
-                <geometry>
-                    <mesh filename="package://dvrk_description/meshes/classic/ecm/insertion_camera_adaptor.stl" />
-                </geometry>
-                <material name="DaVinciDarkGray"/>
-            </visual>
-            <collision>
-                <origin xyz="0 0 0" rpy="0 0 0" />
-                <geometry>
-                    <mesh filename="package://dvrk_description/meshes/classic/ecm/insertion_camera_adaptor.stl" />
+        <link name="${prefix}endoscope_mount_link">
+            <visual>
+                <origin xyz="0 0 0" rpy="0 0 0" />
+                <geometry>
+                    <mesh filename="package://dvrk_description/meshes/classic/ecm/insertion.stl" />
+                </geometry>
+                <material name="DaVinciDarkGray"/>
+            </visual>
+            <collision>
+                <origin xyz="0 0 0" rpy="0 0 0" />
+                <geometry>
+                    <mesh filename="package://dvrk_description/meshes/classic/ecm/insertion.stl" />
                 </geometry>
             </collision>
@@ -167,5 +167,5 @@
         <link name="${prefix}endoscope_link">
             <visual>
-                <origin xyz="0 0 0" rpy="0 0 0" />
+                <origin xyz="0 0 0" rpy="0 0 ${pi/2}" />
                 <geometry>
                     <mesh filename="package://dvrk_description/meshes/classic/ecm/endoscope.stl" />
@@ -174,5 +174,5 @@
             </visual>
             <collision>
-                <origin xyz="0 0 0" rpy="0 0 0" />
+                <origin xyz="0 0 0" rpy="0 0 ${pi/2}" />
                 <geometry>
                     <mesh filename="package://dvrk_description/meshes/classic/ecm/endoscope.stl" />
@@ -240,12 +240,12 @@
             <origin xyz="0.042 -0.086143 0" rpy="${-pi/2} 0 0" />
             <parent link="${prefix}pitch_parallel_end_link" />
-            <child link="${prefix}camera_mount_link" />
+            <child link="${prefix}endoscope_mount_link" />
             <axis xyz="0 0 1" />
             <limit lower="0" upper="0.254193" effort="50" velocity="100" />
         </joint>
-        <joint name="${prefix}camera_roll_joint" type="revolute">
-            <origin xyz="0.0609999999999996 0 0" rpy="0 0 ${pi}" />
-            <parent link="${prefix}camera_mount_link" />
-            <child link="${prefix}camera_link" />
+        <joint name="${prefix}endoscope_roll_joint" type="revolute">
+            <origin xyz="0.0609999999999996 0 0" rpy="0 0 ${pi/2}" />
+            <parent link="${prefix}endoscope_mount_link" />
+            <child link="${prefix}endoscope_link" />
             <axis xyz="0 0 1" />
             <limit lower="${-pi/2}" upper="${pi/2}" effort="1000" velocity="10" />

Commit message: Add ee links

File: urdf/include/classic/ecm.macro.xacro (robot description, xacro)
@@ -272,9 +272,9 @@
         </joint>
         <!-- endoscope tip frame -->
-        <link name="${prefix}tip_link"/>
-        <joint name="${prefix}tip_joint" type="fixed">
+        <link name="${prefix}ee_link"/>
+        <joint name="${prefix}ee_joint" type="fixed">
             <origin xyz="0 0 0.37364" rpy="0 0 0" />
             <parent link="${prefix}endoscope_link" />
-            <child link="${prefix}tip_link" />
+            <child link="${prefix}ee_link" />
             <axis xyz="0 0 0" />
         </joint>

File: urdf/include/classic/tool.macro.xacro (robot description, xacro)
@@ -322,4 +322,11 @@
             <limit lower="0" upper="1" effort="1000" velocity="10" />
         </joint>
+        <!-- End-effector link -->
+        <link name="${prefix}tool_ee_link"/>
+        <joint name="${prefix}tool_ee_joint" type="fixed">
+            <parent link="${prefix}tool_gripper_root_link"/>
+            <child link="${prefix}tool_ee_link"/>
+            <origin xyz="0.005 0 0" rpy="${pi/2} 0 ${pi/2}"/>
+        </joint>
     </xacro:macro>
     <!-- Macro for Cadiere Forceps (cadiere) gripper (8mm) -->
@@ -378,4 +385,11 @@
             <limit lower="0" upper="1" effort="1000" velocity="10" />
         </joint>
+        <!-- End-effector link -->
+        <link name="${prefix}tool_ee_link"/>
+        <joint name="${prefix}tool_ee_joint" type="fixed">
+            <parent link="${prefix}tool_gripper_root_link"/>
+            <child link="${prefix}tool_ee_link"/>
+            <origin xyz="0.005 0 0" rpy="${pi/2} 0 ${pi/2}"/>
+        </joint>
     </xacro:macro>
     <!-- Macro for Round Tip Scissors (rts) gripper (5mm) -->
@@ -434,4 +448,11 @@
             <limit lower="0" upper="1" effort="1000" velocity="10" />
         </joint>
+        <!-- End-effector link -->
+        <link name="${prefix}tool_ee_link"/>
+        <joint name="${prefix}tool_ee_joint" type="fixed">
+            <parent link="${prefix}tool_gripper_root_link"/>
+            <child link="${prefix}tool_ee_link"/>
+            <origin xyz="0.005 0 0" rpy="${pi/2} ${pi} 0"/>
+        </joint>
     </xacro:macro>
 </robot>

File: urdf/include/si/ecm.macro.xacro (robot description, xacro)
@@ -33,5 +33,5 @@
         <link name="${prefix}endoscope_link">
             <visual>
-                <origin xyz="0 0 0" rpy="0 0 0" />
+                <origin xyz="0 0 0" rpy="0 0 ${pi}" />
                 <geometry>
                     <mesh filename="package://dvrk_description/meshes/si/psm_ecm/endoscope.stl"/>
@@ -50,8 +50,15 @@
             <parent link='${prefix}insertion_link'/>
             <child link='${prefix}endoscope_link'/>
-            <origin xyz='0 ${-0.05591} 0' rpy='0 0 ${pi}'/>
+            <origin xyz='0 ${-0.05591} 0' rpy='0 0 0'/>
             <axis xyz='0 0 1'/>
             <limit lower='${-pi}' upper='${pi}' effort='10' velocity='1.0'/>
         </joint>
+        <!-- End-effector link -->
+        <link name="${prefix}ee_link"/>
+        <joint name="${prefix}ee_joint" type="fixed">
+            <parent link="${prefix}endoscope_link"/>
+            <child link="${prefix}ee_link"/>
+            <origin xyz="0 0 0.3976" rpy="0 0 0"/>
+        </joint>
     </xacro:macro>
 </robot>

File: urdf/include/si/tool.macro.xacro (robot description, xacro)
@@ -206,4 +206,11 @@
             <limit lower="0" upper="1" effort="5" velocity="1"/>
         </joint>
+        <!-- End-effector link -->
+        <link name="${prefix}tool_ee_link"/>
+        <joint name="${prefix}tool_ee_joint" type="fixed">
+            <parent link="${prefix}tool_gripper_root_link"/>
+            <child link="${prefix}tool_ee_link"/>
+            <origin xyz="0.005 0 0" rpy="${pi/2} 0 ${pi/2}"/>
+        </joint>
     </xacro:macro>
 </robot>
