Commit message: Fix mismatched tags

File: urdf/include/si/tool.macro.xacro (robot description, xacro)
@@ -80,5 +80,5 @@
                 <material name="DaVinciMetallic"/>
             </visual>
-            <collision></collision>
+            <collision>
                 <origin xyz="0 0 0" rpy="0 0 ${-pi/2}"/>
                 <geometry>
@@ -95,5 +95,5 @@
                 <material name="DaVinciMetallic"/>
             </visual>
-            <collision></collision>
+            <collision>
                 <origin xyz="0 0 0" rpy="${-pi/2} 0 ${-pi/2}"/>
                 <geometry>
