Commit message: fix: correct Si ECM mesh orientation

File: urdf/include/si/ecm.macro.xacro (robot description, xacro)
@@ -33,5 +33,5 @@
         <link name="${prefix}endoscope_link">
             <visual>
-                <origin xyz="0 0 0" rpy="0 0 ${pi}" />
+                <origin xyz="0 0 0" rpy="0 0 0" />
                 <geometry>
                     <mesh filename="package://dvrk_description/meshes/si/psm_ecm/endoscope.stl"/>
