Commit message: Reorganize examples

File: urdf/examples/01_ecm_classic.urdf.xacro (robot description, xacro)
@@ -1,11 +1,17 @@
 <?xml version="1.0" ?>
 <robot name="ecm-classic" xmlns:xacro="http://www.ros.org/wiki/xacro">
-    <!-- Example: ECM Classic -->
+    <!-- Example 01: ECM Classic -->
     <!-- This example spawns an Endoscopic Camera Manipulator (Classic generation) -->
     <xacro:include filename="$(find dvrk_description)/urdf/include/classic/ecm.macro.xacro"/>
     <link name="world"/>
+    <!-- show_RCM
+        * If true, a red sphere will be displayed at the RCM location.
+        * If false, the sphere will be hidden (the default setting).
+    -->
     <xacro:ecm
         prefix=""
+        show_RCM="true"
         parent_link="world"
-        xyz="0 0 0" rpy="0 0 0"/>
+        xyz="0 0 0"
+        rpy="0 0 0"/>
 </robot>

File: urdf/examples/03_mtm_classic.urdf.xacro (robot description, xacro)
@@ -1,11 +1,19 @@
 <?xml version="1.0" ?>
 <robot name="mtm-classic" xmlns:xacro="http://www.ros.org/wiki/xacro">
-    <!-- Example: MTM Classic -->
+    <!-- Example 03: MTM Classic -->
     <!-- This example spawns an Master Tele Manipulator (Classic generation) -->
     <xacro:include filename="$(find dvrk_description)/urdf/include/classic/mtm.macro.xacro"/>
     <link name="world"/>
     <!-- The left hand side MTM -->
-    <xacro:mtm_left prefix="" parent_link="world" xyz="0 0 0" rpy="0 0 0"/>
+    <xacro:mtm_left
+        prefix=""
+        parent_link="world"
+        xyz="0 0 0"
+        rpy="0 0 0"/>
     <!-- The right hand side MTM -->
-    <!-- <xacro:mtm_right prefix="" parent_link="world" xyz="0 0 0" rpy="0 0 0"/> -->
+    <!-- <xacro:mtm_right
+        prefix=""
+        parent_link="world"
+        xyz="0 0 0"
+        rpy="0 0 0"/> -->
 </robot>

File: urdf/examples/05_ecm_si.urdf.xacro (robot description, xacro)
@@ -1,10 +1,15 @@
 <?xml version="1.0" ?>
 <robot name="ecm-si" xmlns:xacro="http://www.ros.org/wiki/xacro">
-    <!-- Example: ECM Si -->
+    <!-- Example 05: ECM Si -->
     <!-- This example spawns an Endoscopic Camera Manipulator (Si generation) -->
     <xacro:include filename="$(find dvrk_description)/urdf/include/si/ecm.macro.xacro"/>
     <link name="world"/>
+    <!-- show_RCM
+        * If true, a red sphere will be displayed at the RCM location.
+        * If false, the sphere will be hidden (the default setting).
+    -->
     <xacro:ecm
         prefix=""
+        show_RCM="true"
         parent_link="world"
         xyz="0 0 0"

File: urdf/examples/06_psm_si.urdf.xacro (robot description, xacro)
@@ -1,13 +1,19 @@
 <?xml version="1.0" ?>
 <robot name="psm-si" xmlns:xacro="https://wiki.ros.org/xacro">
-    <!-- Example: PSM Si -->
+    <!-- Example 06: PSM Si -->
     <!-- This example spawns a Patient Side Manipulator (Si generation) -->
     <xacro:include filename="$(find dvrk_description)/urdf/include/si/psm.macro.xacro"/>
     <link name="world"/>
+    <!-- show_RCM
+        * If true, a red sphere will be displayed at the RCM location.
+        * If false, the sphere will be hidden (the default setting).
+    -->
     <!-- Available tool:
         * lnd_8mm: 8mm large needle driver,
     -->
+    <!-- The Si PSM does not support color modification like Classic PSM -->
     <xacro:psm
         prefix=""
+        show_RCM="true"
         tool="lnd_8mm"
         parent_link="world"

File: urdf/examples/07_tool_si.urdf.xacro (robot description, xacro)
@@ -1,9 +1,13 @@
 <?xml version="1.0" ?>
 <robot name="tool-si" xmlns:xacro="https://wiki.ros.org/xacro">
-    <!-- Example: Tool Si -->
+    <!-- Example 07: Tool Si -->
     <!-- This example spawns the available tool for the Patient Side Manipulator (Si generation) -->
     <xacro:include filename="$(find dvrk_description)/urdf/include/si/tool.macro.xacro"/>
     <link name="world"/>
     <!-- 8mm large needle driver -->
-    <xacro:tool_lnd_8mm prefix="" parent_link="world"/>
+    <xacro:tool_lnd_8mm
+        prefix=""
+        parent_link="world"
+        xyz="0 0 0"
+        rpy="0 0 0"/>
 </robot>

File: urdf/examples/09_patient_cart_si.urdf.xacro (robot description, xacro)
@@ -1,5 +1,5 @@
 <?xml version="1.0" ?>
 <robot name="dvrk-si" xmlns:xacro="http://www.ros.org/wiki/xacro">
-    <!-- Example: Patient Cart Si -->
+    <!-- Example 09: Patient Cart Si -->
     <!-- This example spawns a complete patient cart with three PSMs and an ECM (Si generation) -->
     <xacro:include filename="$(find dvrk_description)/urdf/include/si/suj.macro.xacro"/>
@@ -7,6 +7,7 @@
     <xacro:include filename="$(find dvrk_description)/urdf/include/si/psm.macro.xacro"/>
     <link name="world"/>
+    <xacro:property name="SUJ_PREFIX" value="SUJ_" />
     <xacro:suj
-        prefix="suj_"
+        prefix="${SUJ_PREFIX}"
         parent_link="world"
         include_ecm="true"
@@ -17,17 +18,17 @@
         rpy="0 0 0"/>
     <xacro:ecm
-      prefix="ecm_"
-      parent_link="suj_ecm_mount_link"/>
+        prefix="ECM_"
+        parent_link="${SUJ_PREFIX}ecm_mount_link"/>
     <xacro:psm
-      prefix="psm1_"
-      tool="lnd_8mm"
-      parent_link="suj_psm1_mount_link"/>
+        prefix="PSM1_"
+        tool="lnd_8mm"
+        parent_link="${SUJ_PREFIX}psm1_mount_link"/>
     <xacro:psm
-      prefix="psm2_"
-      tool="lnd_8mm"
-      parent_link="suj_psm2_mount_link"/>
+        prefix="PSM2_"
+        tool="lnd_8mm"
+        parent_link="${SUJ_PREFIX}psm2_mount_link"/>
     <xacro:psm
-      prefix="psm3_"
-      tool="lnd_8mm"
-      parent_link="suj_psm3_mount_link"/>
+        prefix="PSM3_"
+        tool="lnd_8mm"
+        parent_link="${SUJ_PREFIX}psm3_mount_link"/>
 </robot>

File: urdf/examples/10_surgeon_console.urdf.xacro (robot description, xacro)
@@ -1,9 +1,13 @@
 <?xml version="1.0" ?>
 <robot name="surgeon_console" xmlns:xacro="http://www.ros.org/wiki/xacro">
-    <!-- Example: Surgeon Console -->
+    <!-- Example 10: Surgeon Console -->
     <!-- This example spawns a Surgeon Console -->
     <!-- The Classic and Si generations share the same surgeon console -->
     <xacro:include filename="$(find dvrk_description)/urdf/include/classic/mtm.macro.xacro"/>
     <link name="world"/>
-    <xacro:surgeon_console prefix="" parent_link="world" xyz="0 0 0" rpy="0 0 0"/>
+    <xacro:surgeon_console
+        prefix=""
+        parent_link="world"
+        xyz="0 0 0"
+        rpy="0 0 0"/>
 </robot>
