Commit message: Add generation suffix to marcos

File: urdf/examples/01_ecm_classic.urdf.xacro (robot description, xacro)
@@ -9,5 +9,5 @@
         * If false, the sphere will be hidden (the default setting).
     -->
-    <xacro:ecm
+    <xacro:ecm_classic
         prefix=""
         show_RCM="true"

File: urdf/examples/02_psm_classic.urdf.xacro (robot description, xacro)
@@ -20,7 +20,7 @@
         * rts_5mm: 5mm round tip scissors.
     -->
-    <xacro:psm
+    <xacro:psm_classic
         prefix=""
-        color="DavinciOrange"
+        color="DaVinciOrange"
         show_RCM="true"
         tool="sca_8mm"

File: urdf/examples/03_mtm_classic.urdf.xacro (robot description, xacro)
@@ -6,5 +6,5 @@
     <link name="world"/>
     <!-- The left hand side MTM -->
-    <xacro:mtm_left
+    <xacro:mtm_left_classic
         prefix=""
         parent_link="world"
@@ -12,5 +12,5 @@
         rpy="0 0 0"/>
     <!-- The right hand side MTM -->
-    <!-- <xacro:mtm_right
+    <!-- <xacro:mtm_right_classic
         prefix=""
         parent_link="world"

File: urdf/examples/04_tool_classic.urdf.xacro (robot description, xacro)
@@ -6,17 +6,20 @@
     <link name="world"/>
     <!-- 8mm small clip applier -->
-    <xacro:tool_sca_8mm
+    <xacro:tool_sca_8mm_classic
         prefix="sca_"
         parent_link="world"
-        xyz="0 0 0"/>
+        xyz="0 0 0"
+        rpy="0 0 0"/>
     <!-- 8mm cadiere forceps -->
-    <xacro:tool_cadiere_8mm
+    <xacro:tool_cadiere_8mm_classic
         prefix="cadiere_"
         parent_link="world"
-        xyz="-0.3 0 0"/>
+        xyz="-0.3 0 0"
+        rpy="0 0 0"/>
     <!-- 5mm round tip scissors -->
-    <xacro:tool_rts_5mm
+    <xacro:tool_rts_5mm_classic
         prefix="rts_"
         parent_link="world"
-        xyz="0.3 0 0"/>
+        xyz="0.3 0 0"
+        rpy="0 0 0"/>
 </robot>

File: urdf/examples/05_ecm_si.urdf.xacro (robot description, xacro)
@@ -9,5 +9,5 @@
         * If false, the sphere will be hidden (the default setting).
     -->
-    <xacro:ecm
+    <xacro:ecm_si
         prefix=""
         show_RCM="true"

File: urdf/examples/06_psm_si.urdf.xacro (robot description, xacro)
@@ -13,5 +13,5 @@
     -->
     <!-- The Si PSM does not support color modification like Classic PSM -->
-    <xacro:psm
+    <xacro:psm_si
         prefix=""
         show_RCM="true"

File: urdf/examples/07_tool_si.urdf.xacro (robot description, xacro)
@@ -6,5 +6,5 @@
     <link name="world"/>
     <!-- 8mm large needle driver -->
-    <xacro:tool_lnd_8mm
+    <xacro:tool_lnd_8mm_si
         prefix=""
         parent_link="world"

File: urdf/examples/08_patient_cart_classic.urdf.xacro (robot description, xacro)
@@ -8,5 +8,5 @@
     <link name="world"/>
     <xacro:property name="SUJ_PREFIX" value="SUJ_" />
-    <xacro:suj
+    <xacro:suj_classic
         prefix="${SUJ_PREFIX}"
         parent_link="world"
@@ -17,18 +17,18 @@
         xyz="0 0 0"
         rpy="0 0 0"/>
-    <xacro:ecm
+    <xacro:ecm_classic
         prefix="ECM_"
         parent_link="${SUJ_PREFIX}ecm_mount_link"/>
-    <xacro:psm
+    <xacro:psm_classic
         prefix="PSM1_"
         tool="rts_5mm"
         color="DaVinciOrange"
         parent_link="${SUJ_PREFIX}psm1_mount_link"/>
-    <xacro:psm
+    <xacro:psm_classic
         prefix="PSM2_"
         tool="cadiere_8mm"
         color="DaVinciLightBlue"
         parent_link="${SUJ_PREFIX}psm2_mount_link"/>
-    <xacro:psm
+    <xacro:psm_classic
         prefix="PSM3_"
         tool="sca_8mm"

File: urdf/examples/09_patient_cart_si.urdf.xacro (robot description, xacro)
@@ -8,5 +8,5 @@
     <link name="world"/>
     <xacro:property name="SUJ_PREFIX" value="SUJ_" />
-    <xacro:suj
+    <xacro:suj_si
         prefix="${SUJ_PREFIX}"
         parent_link="world"
@@ -17,16 +17,16 @@
         xyz="0 0 0"
         rpy="0 0 0"/>
-    <xacro:ecm
+    <xacro:ecm_si
         prefix="ECM_"
         parent_link="${SUJ_PREFIX}ecm_mount_link"/>
-    <xacro:psm
+    <xacro:psm_si
         prefix="PSM1_"
         tool="lnd_8mm"
         parent_link="${SUJ_PREFIX}psm1_mount_link"/>
-    <xacro:psm
+    <xacro:psm_si
         prefix="PSM2_"
         tool="lnd_8mm"
         parent_link="${SUJ_PREFIX}psm2_mount_link"/>
-    <xacro:psm
+    <xacro:psm_si
         prefix="PSM3_"
         tool="lnd_8mm"

File: urdf/examples/10_surgeon_console.urdf.xacro (robot description, xacro)
@@ -6,5 +6,5 @@
     <xacro:include filename="$(find dvrk_description)/urdf/include/classic/mtm.macro.xacro"/>
     <link name="world"/>
-    <xacro:surgeon_console
+    <xacro:surgeon_console_classic
         prefix=""
         parent_link="world"

File: urdf/include/classic/ecm.macro.xacro (robot description, xacro)
@@ -3,5 +3,5 @@
     <xacro:include filename="$(find dvrk_description)/urdf/include/colors.xacro"/>
     <!-- Macro for da Vinci Endoscope Camera Manipulator (ecm) -->
-    <xacro:macro name="ecm" params="prefix show_RCM:='false' parent_link xyz:='0 0 0' rpy:='0 0 0'">
+    <xacro:macro name="ecm_classic" params="prefix show_RCM:='false' parent_link xyz:='0 0 0' rpy:='0 0 0'">
         <!-- ECM links -->
         <link name="${prefix}base_link">

File: urdf/include/classic/mtm.macro.xacro (robot description, xacro)
@@ -3,5 +3,5 @@
     <xacro:include filename="$(find dvrk_description)/urdf/include/colors.xacro"/>
     <!-- Macro for the surgeon console -->
-    <xacro:macro name="surgeon_console" params="prefix parent_link xyz:='0.0 0.0 0.0' rpy:='0.0 0.0 0.0'">
+    <xacro:macro name="surgeon_console_classic" params="prefix parent_link xyz:='0.0 0.0 0.0' rpy:='0.0 0.0 0.0'">
         <link name="${prefix}base_link"/>
         <joint name="${prefix}base_joint" type="fixed">
@@ -10,19 +10,37 @@
             <origin xyz="${xyz}" rpy="${rpy}"/>
         </joint>
-        <xacro:mtm_left prefix="${prefix}MTML_" parent_link="${prefix}base_link" xyz="0 -0.25 1" />
-        <xacro:mtm_right prefix="${prefix}MTMR_" parent_link="${prefix}base_link" xyz="0 0.25 1" />
+        <xacro:mtm_left_classic
+            prefix="${prefix}MTML_"
+            parent_link="${prefix}base_link"
+            xyz="0 -0.25 1" />
+        <xacro:mtm_right_classic
+            prefix="${prefix}MTMR_"
+            parent_link="${prefix}base_link"
+            xyz="0 0.25 1" />
     </xacro:macro>
     <!-- Macro for a complete MTM with the left wrist -->
-    <xacro:macro name="mtm_left" params="prefix parent_link xyz:='0.0 0.0 0.0' rpy:='0.0 0.0 0.0'">
-        <xacro:mtm_arm prefix="${prefix}" parent_link="${parent_link}" xyz="${xyz}" rpy="${rpy}"/>
-        <xacro:mtm_wrist_left prefix="${prefix}" parent_link="${prefix}wrist_mount_link"/>
+    <xacro:macro name="mtm_left_classic" params="prefix parent_link xyz:='0.0 0.0 0.0' rpy:='0.0 0.0 0.0'">
+        <xacro:mtm_arm_classic
+            prefix="${prefix}"
+            parent_link="${parent_link}"
+            xyz="${xyz}"
+            rpy="${rpy}"/>
+        <xacro:mtm_wrist_left_classic
+            prefix="${prefix}"
+            parent_link="${prefix}wrist_mount_link"/>
     </xacro:macro>
     <!-- Macro for a complete MTM with the right wrist -->
-    <xacro:macro name="mtm_right" params="prefix parent_link xyz:='0.0 0.0 0.0' rpy:='0.0 0.0 0.0'">
-        <xacro:mtm_arm prefix="${prefix}" parent_link="${parent_link}" xyz="${xyz}" rpy="${rpy}"/>
-        <xacro:mtm_wrist_right prefix="${prefix}" parent_link="${prefix}wrist_mount_link"/>
+    <xacro:macro name="mtm_right_classic" params="prefix parent_link xyz:='0.0 0.0 0.0' rpy:='0.0 0.0 0.0'">
+        <xacro:mtm_arm_classic
+            prefix="${prefix}"
+            parent_link="${parent_link}"
+            xyz="${xyz}"
+            rpy="${rpy}"/>
+        <xacro:mtm_wrist_right_classic
+            prefix="${prefix}"
+            parent_link="${prefix}wrist_mount_link"/>
     </xacro:macro>
     <!-- Macro for MTM arm without wrist -->
-    <xacro:macro name="mtm_arm" params="prefix parent_link xyz:='0.0 0.0 0.0' rpy:='0.0 0.0 0.0'">
+    <xacro:macro name="mtm_arm_classic" params="prefix parent_link xyz:='0.0 0.0 0.0' rpy:='0.0 0.0 0.0'">
         <!-- MTM arm links -->
         <link name="${prefix}base_link">
@@ -194,5 +212,5 @@
     </xacro:macro>
     <!-- Macro for MTM left wrist -->
-    <xacro:macro name="mtm_wrist_left" params="prefix parent_link xyz:='0.0 0.0 0.0' rpy:='0.0 0.0 0.0'">
+    <xacro:macro name="mtm_wrist_left_classic" params="prefix parent_link xyz:='0.0 0.0 0.0' rpy:='0.0 0.0 0.0'">
         <!-- MTM wrist left links -->
         <link name="${prefix}wrist_yaw1_link">
@@ -305,5 +323,5 @@
     </xacro:macro>
     <!-- Macro for MTM right wrist -->
-    <xacro:macro name="mtm_wrist_right" params="prefix parent_link xyz:='0.0 0.0 0.0' rpy:='0.0 0.0 0.0'">
+    <xacro:macro name="mtm_wrist_right_classic" params="prefix parent_link xyz:='0.0 0.0 0.0' rpy:='0.0 0.0 0.0'">
         <!-- MTM wrist right links -->
         <link name="${prefix}wrist_yaw1_link">

File: urdf/include/classic/psm.macro.xacro (robot description, xacro)
@@ -4,6 +4,6 @@
     <xacro:include filename="$(find dvrk_description)/urdf/include/classic/tool.macro.xacro"/>
     <!-- Macro for a complete PSM with tool -->
-    <xacro:macro name="psm" params="prefix color:='DaVinciOrange' show_RCM:='false' tool:='sca_8mm' parent_link xyz:='0 0 0' rpy:='0 0 0'">
-        <xacro:psm_arm
+    <xacro:macro name="psm_classic" params="prefix color:='DaVinciOrange' show_RCM:='false' tool:='sca_8mm' parent_link xyz:='0 0 0' rpy:='0 0 0'">
+        <xacro:psm_arm_classic
             prefix="${prefix}"
             color="${color}"
@@ -14,5 +14,5 @@
         <!-- 8mm Small Clip Applier -->
         <xacro:if value="${tool == 'sca_8mm'}">
-            <xacro:tool_sca_8mm
+            <xacro:tool_sca_8mm_classic
                 prefix="${prefix}"
                 parent_link="${prefix}tool_mount_link"/>
@@ -20,5 +20,5 @@
         <!-- 8mm Cadiere Forceps -->
         <xacro:if value="${tool == 'cadiere_8mm'}">
-            <xacro:tool_cadiere_8mm
+            <xacro:tool_cadiere_8mm_classic
                 prefix="${prefix}"
                 parent_link="${prefix}tool_mount_link"/>
@@ -26,5 +26,5 @@
         <!-- 5mm Round Tip Scissors -->
         <xacro:if value="${tool == 'rts_5mm'}">
-            <xacro:tool_rts_5mm
+            <xacro:tool_rts_5mm_classic
                 prefix="${prefix}"
                 parent_link="${prefix}tool_mount_link"/>
@@ -32,5 +32,5 @@
     </xacro:macro>
     <!-- Macro for a PSM arm without tool -->
-    <xacro:macro name="psm_arm" params="prefix color:='DaVinciOrange' show_RCM:='false' parent_link xyz:='0 0 0' rpy:='0 0 0'">
+    <xacro:macro name="psm_arm_classic" params="prefix color:='DaVinciOrange' show_RCM:='false' parent_link xyz:='0 0 0' rpy:='0 0 0'">
         <!-- PSM arm links -->
         <link name="${prefix}base_link">

File: urdf/include/classic/suj.macro.xacro (robot description, xacro)
@@ -3,21 +3,37 @@
     <xacro:include filename="$(find dvrk_description)/urdf/include/colors.xacro"/>
     <!-- Macro for the complete SUJ -->
-    <xacro:macro name='suj' params="prefix include_ecm:=false include_psm1:=false include_psm2:=false include_psm3:=false parent_link xyz:='0 0 0' rpy:='0 0 0'">
-        <xacro:suj_tower prefix="${prefix}" parent_link="${parent_link}" xyz="${xyz}" rpy="${rpy}"/>
+    <xacro:macro name='suj_classic' params="prefix include_ecm:=false include_psm1:=false include_psm2:=false include_psm3:=false parent_link xyz:='0 0 0' rpy:='0 0 0'">
+        <xacro:suj_tower_classic
+            prefix="${prefix}"
+            parent_link="${parent_link}"
+            xyz="${xyz}"
+            rpy="${rpy}"/>
         <xacro:if value="${include_ecm}">
-            <xacro:suj_arm type="ecm" prefix="${prefix}ecm_" parent_link="${prefix}suj_arm_ecm_mount_link"/>
+            <xacro:suj_arm_classic
+                type="ecm"
+                prefix="${prefix}ecm_"
+                parent_link="${prefix}suj_arm_ecm_mount_link"/>
         </xacro:if>
         <xacro:if value="${include_psm1}">
-            <xacro:suj_arm type="psm1" prefix="${prefix}psm1_" parent_link="${prefix}suj_arm_psm1_mount_link"/>
+            <xacro:suj_arm_classic
+                type="psm1"
+                prefix="${prefix}psm1_"
+                parent_link="${prefix}suj_arm_psm1_mount_link"/>
         </xacro:if>
         <xacro:if value="${include_psm2}">
-            <xacro:suj_arm type="psm2" prefix="${prefix}psm2_" parent_link="${prefix}suj_arm_psm2_mount_link"/>
+            <xacro:suj_arm_classic
+                type="psm2"
+                prefix="${prefix}psm2_"
+                parent_link="${prefix}suj_arm_psm2_mount_link"/>
         </xacro:if>
         <xacro:if value="${include_psm3}">
-            <xacro:suj_arm type="psm3" prefix="${prefix}psm3_" parent_link="${prefix}suj_arm_psm3_mount_link"/>
+            <xacro:suj_arm_classic
+                type="psm3"
+                prefix="${prefix}psm3_"
+                parent_link="${prefix}suj_arm_psm3_mount_link"/>
         </xacro:if>
     </xacro:macro>
     <!-- Macro for the SUJ tower -->
-    <xacro:macro name='suj_tower' params="prefix parent_link xyz:='0 0 0' rpy:='0 0 0'">
+    <xacro:macro name='suj_tower_classic' params="prefix parent_link xyz:='0 0 0' rpy:='0 0 0'">
         <link name="${prefix}base_link"/>
         <link name="${prefix}tower_link">
@@ -77,20 +93,32 @@
     </xacro:macro>
     <!-- Macro for the SUJ arm -->
-    <xacro:macro name='suj_arm' params="prefix type parent_link xyz:='0 0 0' rpy:='0 0 0'">
+    <xacro:macro name='suj_arm_classic' params="prefix type parent_link xyz:='0 0 0' rpy:='0 0 0'">
         <!-- ECM -->
         <xacro:if value="${type == 'ecm'}">
-            <xacro:suj_arm_ecm prefix="${prefix}" parent_link="${parent_link}" xyz="${xyz}" rpy="${rpy}"/>
+            <xacro:suj_arm_ecm_classic
+                prefix="${prefix}"
+                parent_link="${parent_link}"
+                xyz="${xyz}"
+                rpy="${rpy}"/>
         </xacro:if>
         <!-- PSM1 or PSM2 -->
         <xacro:if value="${type == 'psm1' or type == 'psm2'}">
-            <xacro:suj_arm_psm12 prefix="${prefix}" parent_link="${parent_link}" xyz="${xyz}" rpy="${rpy}"/>
+            <xacro:suj_arm_psm12_classic
+                prefix="${prefix}"
+                parent_link="${parent_link}"
+                xyz="${xyz}"
+                rpy="${rpy}"/>
         </xacro:if>
         <!-- PSM3 -->
         <xacro:if value="${type == 'psm3'}">
-            <xacro:suj_arm_psm3 prefix="${prefix}" parent_link="${parent_link}" xyz="${xyz}" rpy="${rpy}"/>
+            <xacro:suj_arm_psm3_classic
+                prefix="${prefix}"
+                parent_link="${parent_link}"
+                xyz="${xyz}"
+                rpy="${rpy}"/>
         </xacro:if>
     </xacro:macro>
     <!-- Macro for the SUJ arm for mounting the ECM -->
-    <xacro:macro name='suj_arm_ecm' params="prefix parent_link xyz:='0 0 0' rpy:='0 0 0'">
+    <xacro:macro name='suj_arm_ecm_classic' params="prefix parent_link xyz:='0 0 0' rpy:='0 0 0'">
         <link name="${prefix}lift_link">
             <visual>
@@ -209,5 +237,5 @@
     </xacro:macro>
     <!-- Macro for the SUJ arm for mounting the PSM1 and PSM2 -->
-    <xacro:macro name='suj_arm_psm12' params="prefix parent_link xyz:='0 0 0' rpy:='0 0 0'">
+    <xacro:macro name='suj_arm_psm12_classic' params="prefix parent_link xyz:='0 0 0' rpy:='0 0 0'">
         <link name="${prefix}lift_link">
             <visual>
@@ -355,5 +383,5 @@
     </xacro:macro>
     <!-- Macro for the SUJ arm for mounting the PSM3 -->
-    <xacro:macro name='suj_arm_psm3' params="prefix parent_link xyz:='0 0 0' rpy:='0 0 0'">
+    <xacro:macro name='suj_arm_psm3_classic' params="prefix parent_link xyz:='0 0 0' rpy:='0 0 0'">
         <link name="${prefix}lift_link">
             <visual>

File: urdf/include/classic/tool.macro.xacro (robot description, xacro)
@@ -3,6 +3,6 @@
     <xacro:include filename="$(find dvrk_description)/urdf/include/colors.xacro"/>
     <!-- Macro for the 8mm Small Clip Applier (sca) tool -->
-    <xacro:macro name="tool_sca_8mm" params="prefix parent_link xyz:='0 0 0' rpy:='0 0 0'">
-        <xacro:tool_shaft
+    <xacro:macro name="tool_sca_8mm_classic" params="prefix parent_link xyz:='0 0 0' rpy:='0 0 0'">
+        <xacro:tool_shaft_classic
             prefix="${prefix}"
             diameter="8mm"
@@ -10,14 +10,14 @@
             xyz="${xyz}"
             rpy="${rpy}"/>
-        <xacro:tool_wrist_8mm
+        <xacro:tool_wrist_8mm_classic
             prefix="${prefix}"
             parent_link="${prefix}tool_wrist_mount_link"/>
-        <xacro:tool_gripper_sca_8mm
+        <xacro:tool_gripper_sca_8mm_classic
             prefix="${prefix}"
             parent_link="${prefix}tool_gripper_mount_link"/>
     </xacro:macro>
     <!-- Macro for the 8mm Cadiere Forceps (cadiere) tool -->
-    <xacro:macro name="tool_cadiere_8mm" params="prefix parent_link xyz:='0 0 0' rpy:='0 0 0'">
-        <xacro:tool_shaft
+    <xacro:macro name="tool_cadiere_8mm_classic" params="prefix parent_link xyz:='0 0 0' rpy:='0 0 0'">
+        <xacro:tool_shaft_classic
             prefix="${prefix}"
             diameter="8mm"
@@ -25,14 +25,14 @@
             xyz="${xyz}"
             rpy="${rpy}"/>
-        <xacro:tool_wrist_8mm
+        <xacro:tool_wrist_8mm_classic
             prefix="${prefix}"
             parent_link="${prefix}tool_wrist_mount_link"/>
-        <xacro:tool_gripper_cadiere_8mm
+        <xacro:tool_gripper_cadiere_8mm_classic
             prefix="${prefix}"
             parent_link="${prefix}tool_gripper_mount_link"/>
     </xacro:macro>
     <!-- Macro for the 5mm Round Tip Scissors (rts) tool -->
-    <xacro:macro name="tool_rts_5mm" params="prefix parent_link xyz:='0 0 0' rpy:='0 0 0'">
-        <xacro:tool_shaft
+    <xacro:macro name="tool_rts_5mm_classic" params="prefix parent_link xyz:='0 0 0' rpy:='0 0 0'">
+        <xacro:tool_shaft_classic
             prefix="${prefix}"
             diameter="5mm"
@@ -40,13 +40,13 @@
             xyz="${xyz}"
             rpy="${rpy}"/>
-        <xacro:tool_wrist_5mm
+        <xacro:tool_wrist_5mm_classic
             prefix="${prefix}"
             parent_link="${prefix}tool_wrist_mount_link"/>
-        <xacro:tool_gripper_rts_5mm
+        <xacro:tool_gripper_rts_5mm_classic
             prefix="${prefix}"
             parent_link="${prefix}tool_gripper_mount_link"/>
     </xacro:macro>
     <!-- Macro for tool shaft (8mm and 5mm)  -->
-    <xacro:macro name="tool_shaft" params="prefix diameter parent_link xyz:='0 0 0' rpy:='0 0 0'">
+    <xacro:macro name="tool_shaft_classic" params="prefix diameter parent_link xyz:='0 0 0' rpy:='0 0 0'">
         <link name="${prefix}tool_base_link">
             <visual>
@@ -98,5 +98,5 @@
     </xacro:macro>
     <!-- Macro for tool wrist (8mm) -->
-    <xacro:macro name="tool_wrist_8mm" params="prefix parent_link xyz:='0 0 0' rpy:='0 0 0'">
+    <xacro:macro name="tool_wrist_8mm_classic" params="prefix parent_link xyz:='0 0 0' rpy:='0 0 0'">
         <!-- 8mm wrist links -->
         <link name="${prefix}tool_wrist_roll_link">
@@ -176,5 +176,5 @@
     </xacro:macro>
     <!-- Macro for tool wrist (5mm) -->
-    <xacro:macro name="tool_wrist_5mm" params="prefix parent_link xyz:='0 0 0' rpy:='0 0 0'">
+    <xacro:macro name="tool_wrist_5mm_classic" params="prefix parent_link xyz:='0 0 0' rpy:='0 0 0'">
         <!-- 5mm wrist links -->
         <link name="${prefix}tool_wrist_roll_link">
@@ -268,5 +268,5 @@
     </xacro:macro>
     <!-- Macro for Small Clip Applier (sca) gripper (8mm) -->
-    <xacro:macro name="tool_gripper_sca_8mm" params="prefix parent_link xyz:='0 0 0' rpy:='0 0 0'">
+    <xacro:macro name="tool_gripper_sca_8mm_classic" params="prefix parent_link xyz:='0 0 0' rpy:='0 0 0'">
         <!-- sca gripper links -->
         <link name="${prefix}tool_gripper_root_link"/>
@@ -324,5 +324,5 @@
     </xacro:macro>
     <!-- Macro for Cadiere Forceps (cadiere) gripper (8mm) -->
-    <xacro:macro name="tool_gripper_cadiere_8mm" params="prefix parent_link xyz:='0 0 0' rpy:='0 0 0'">
+    <xacro:macro name="tool_gripper_cadiere_8mm_classic" params="prefix parent_link xyz:='0 0 0' rpy:='0 0 0'">
         <!-- cadiere gripper links -->
         <link name="${prefix}tool_gripper_root_link"/>
@@ -380,5 +380,5 @@
     </xacro:macro>
     <!-- Macro for Round Tip Scissors (rts) gripper (5mm) -->
-    <xacro:macro name="tool_gripper_rts_5mm" params="prefix parent_link xyz:='0 0 0' rpy:='0 0 0'">
+    <xacro:macro name="tool_gripper_rts_5mm_classic" params="prefix parent_link xyz:='0 0 0' rpy:='0 0 0'">
         <!-- rts gripper links -->
         <link name="${prefix}tool_gripper_root_link"/>

File: urdf/include/si/ecm.macro.xacro (robot description, xacro)
@@ -4,6 +4,6 @@
     <xacro:include filename="$(find dvrk_description)/urdf/include/si/psm.macro.xacro"/>
     <!-- Macro for an ECM -->
-    <xacro:macro name="ecm" params="prefix show_RCM:='false' parent_link xyz:='0 0 0' rpy:= '0 0 0'">
-        <xacro:psm_ecm_body
+    <xacro:macro name="ecm_si" params="prefix show_RCM:='false' parent_link xyz:='0 0 0' rpy:= '0 0 0'">
+        <xacro:psm_ecm_body_si
             prefix='${prefix}'
             show_RCM='${show_RCM}'

File: urdf/include/si/psm.macro.xacro (robot description, xacro)
@@ -4,6 +4,6 @@
     <xacro:include filename="$(find dvrk_description)/urdf/include/si/tool.macro.xacro"/>
     <!-- Macro for a PSM with tool -->
-    <xacro:macro name="psm" params="prefix show_RCM:='false' tool:='lnd_8mm' parent_link xyz:='0 0 0' rpy:= '0 0 0'">
-        <xacro:psm_arm
+    <xacro:macro name="psm_si" params="prefix show_RCM:='false' tool:='lnd_8mm' parent_link xyz:='0 0 0' rpy:= '0 0 0'">
+        <xacro:psm_arm_si
             prefix='${prefix}'
             show_RCM='${show_RCM}'
@@ -12,5 +12,5 @@
             rpy='${rpy}'/>
         <xacro:if value="${tool == 'lnd_8mm'}">
-            <xacro:tool_lnd_8mm
+            <xacro:tool_lnd_8mm_si
                 prefix='${prefix}'
                 parent_link='${prefix}tool_mount_link'/>
@@ -18,6 +18,6 @@
     </xacro:macro>
     <!-- Macro for a PSM without tool -->
-    <xacro:macro name="psm_arm" params="prefix show_RCM:='false' parent_link xyz:='0 0 0' rpy:= '0 0 0'">
-        <xacro:psm_ecm_body
+    <xacro:macro name="psm_arm_si" params="prefix show_RCM:='false' parent_link xyz:='0 0 0' rpy:= '0 0 0'">
+        <xacro:psm_ecm_body_si
             prefix='${prefix}'
             show_RCM='${show_RCM}'
@@ -61,5 +61,5 @@
     </xacro:macro>
     <!-- Macro for the PSM/ECM main structure -->
-    <xacro:macro name="psm_ecm_body" params="prefix show_RCM:='false' parent_link xyz:='0 0 0' rpy:= '0 0 0'">
+    <xacro:macro name="psm_ecm_body_si" params="prefix show_RCM:='false' parent_link xyz:='0 0 0' rpy:= '0 0 0'">
         <link name='${prefix}base_link'>
             <visual>
